File: PwrRails.sch (KiCad schematic (older format))
At the start: 99 parts, among them IC1 ATMEGA8-AI, P1 CONN_01X02, P10 CONN_01X02, P11 CONN_01X03, P12 PR 5V, P13 PR 5V, P2 PR 5V, P3 CONN_01X02, P4 CONN_01X05, P5 CONN_01X01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

Commit message: 12V Seite fast fertig
Connections:
- net Switch_5V: no longer C27.1, L3.1, U4.10 (SW), U4.11 (SW)
- net VFB_5V: no longer C29.1, R31.2, R34.1, U4.2 (VFB)
- net Switch_12V: now reaches C12.2, L2.1, U2.3 (PH)
- new net Switch_3V: C27.1, L3.1, U4.10 (SW), U4.11 (SW)
- new net VFB_3V: C29.1, R31.2, R34.1, U4.2 (VFB)
Changed lines of the file:
@@
 $EndComp
 Text Label 13575 5750 0    60   ~ 0
-Switch_5V
+Switch_3V
 $Comp
 L GND #PWR061
@@
 $EndComp
 Text Label 10900 6175 0    60   ~ 0
-VFB_5V
+VFB_3V
 Text GLabel 15225 7200 3    60   Output ~ 0
 AGND
@@
 Wire Wire Line
 	14425 8400 14425 8375
+Text Label 13275 3875 1    60   ~ 0
+Switch_12V
 $EndSCHEMATC

Commit message: PCB quasi fertig!
Parts:
- added C33: 1µ, Capacitors_SMD:C_0805, symbol C
- added Q1: Q_PMOS_GSD, TO_SOT_Packages_SMD:SOT-23, symbol Q_PMOS_GSD
- added R40, R41, R42, R43: R, Resistors_SMD:R_0603, symbol R
- added U5: LM293, SMD_Packages:SOIC-8-N, symbol LM293
- added U6: NCP51460, TO_SOT_Packages_SMD:SOT-23, symbol NCP51460
- added X1: CRYSTAL_SMD, Toni:CerOsc_3,2x1,3, symbol CRYSTAL_SMD
- C16, C2: footprint Capacitors_SMD:C_1206 -> Capacitors_SMD:C_1210
- L1: footprint Inductors_NEOSID:Neosid_Inductor_SM-NE127 -> Sven:Z_Borus_SRN8040
- L3: footprint Inductors_NEOSID:Neosid_Inductor_SM-NE127 -> Sven:Z_Coilcraft_XFL4020
- P6: footprint Socket_Strips:Socket_Strip_Straight_1x06 -> Socket_Strips:Socket_Strip_Straight_2x03
Connections:
- net +12V: now also R22.2
- net +3V3: now also Q1.2 (S), R40.2, R41.2, U5.8 (V+); no longer P8.5 (P5), R22.2
- net +5V: now also C33.1, U6.1 (Vin)
- net AGND: no longer D1.2 (A), D2.2 (A), D3.2 (A), D4.2 (A), D5.2 (A), D6.2 (A)
- net GND: now also D1.2 (A), D2.2 (A), D3.2 (A), D4.2 (A), D5.2 (A), D6.2 (A), C33.2, U5.4 (V-), U6.3 (GND), X1.3 (case)
- net at IC1.7 (PB6(XTAL1/TOSC1)): now also X1.1
- net at IC1.8 (PB7(XTAL2/TOSC2)): now also X1.2
- new net: Q1.1 (G), R40.1, R43.1, U5.1
- new net: U5.2 (_), U6.2 (Vout)
- new net: R42.1, R43.2, U5.3 (+)
- new net: R41.1, R42.2
- new net Switched_3V3: P8.5 (P5), Q1.3 (D)

Commit message: Bohrungen hinzugefügt.
Parts:
- added P14: CONN_01X01, Socket_Strips:Socket_Strip_Straight_1x01, symbol CONN_01X01
Connections:
- net GND: now also P14.1 (P1)
